File: pcb_design/kicad_schematics/schematics.kicad_sch (KiCad schematic)
At the start: 29 parts, among them J10 LED-HSF08A/B, J11 BUTTON-HS-KEY1B, J6 PICKIT, J7 I2C_Communication_Protocol, J8 M22-2510205, J9 SG90, U1 PIC24FJ64GA702-I_SO, U2 ESP8266-01_ESP-01, U3 LM1117LD-3.3, Y2 16MHz crystal

Commit message: 13.1.25, dodani footprinti i inicijalna sema pcba
Parts:
- C1, C11, C13, C3, C5: footprint C_Ceramic-100nF:C0402 -> C_Ceramic_100n:C0402
- C10, C9: footprint C_Polarized_Tantalum-10uF:CAPPC3528X210N -> C_Polarized_Tantalum-10u:CAPPC3528X210N
- C12, C2, C4, C6: footprint C_Ceramic-10uF:C0805 -> C_Ceramic_100n:C0402
- C14: footprint C0805 -> C_Ceramic_100n:C0402
- C15, C16: footprint CAPC2012X145N -> C_Ceramic_100n:C0402
- C7, C8: value 10u -> 0.1u; footprint C_Polarized_Tantalum-10uF:CAPPC3528X210N -> C_Polarized_Tantalum-10u:CAPPC3528X210N
- J10, J11, J9: footprint HDRV3W60P0X200_1X3_600X200X525P -> 3_PIN_MALE:HDRV3W60P0X200_1X3_600X200X525P
- J6, J7: footprint HDRV5W64P0X254_1X5_1270X254X610P -> 5_PIN_MALE:HDRV5W64P0X254_1X5_1270X254X610P
- J8: footprint 2_pin_Male:HDRV2W60P0X200_1X2_400X200X525P -> 2_PIN_MALE:HDRV2W60P0X200_1X2_400X200X525P
- JP1: footprint (none) -> 2_PIN_MALE:HDRV2W60P0X200_1X2_400X200X525P
- R1, R2: footprint (none) -> Resistor_SMD:R_0805_2012Metric_Pad1.20x1.40mm_HandSolder
- U1: footprint Microcontroller-PIC24FJ64GA702-I_SO:SOIC127P1030X265-28N -> PIC:SOIC127P1030X265-28N
- U2: footprint ESP8266-01_ESP-01:XCVR_ESP8266-01_ESP-01 -> ESP8266EX:XCVR_ESP8266-01_ESP-01
- Y2: footprint 830108288709 -> Crystal16MHZ:830108288709
Changed lines of the file:
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@@
 			)
 		)
-		(property "Footprint" "Microcontroller-PIC24FJ64GA702-I_SO:SOIC127P1030X265-28N"
+		(property "Footprint" "PIC:SOIC127P1030X265-28N"
 			(at 158.75 201.6 0)
 			(effects
@@
 			)
 		)
-		(property "Footprint" "C_Ceramic-100nF:C0402"
+		(property "Footprint" "C_Ceramic_100n:C0402"
 			(at -0.94 124.46 0)
 			(effects
@@
 			)
 		)
-		(property "Footprint" "HDRV5W64P0X254_1X5_1270X254X610P"
+		(property "Footprint" "5_PIN_MALE:HDRV5W64P0X254_1X5_1270X254X610P"
 			(at 148.59 134.29 0)
 			(effects
@@
 			)
 		)
-		(property "Footprint" "C_Ceramic-10uF:C0805"
+		(property "Footprint" "C_Ceramic_100n:C0402"
 			(at 366.7 114.3 0)
 			(effects
@@
 			)
 		)
-		(property "Footprint" "C_Ceramic-100nF:C0402"
+		(property "Footprint" "C_Ceramic_100n:C0402"
 			(at 272.72 95.25 0)
 			(effects
@@
 			)
 		)
-		(property "Footprint" ""
+		(property "Footprint" "Resistor_SMD:R_0805_2012Metric_Pad1.20x1.40mm_HandSolder"
 			(at 116.84 108.458 90)
 			(effects
@@
 			)
 		)
-		(property "Footprint" "C_Ceramic-100nF:C0402"
+		(property "Footprint" "C_Ceramic_100n:C0402"
 			(at 205.41 140.97 0)
 			(effects
@@
 			)
 		)
-		(property "Footprint" "HDRV3W60P0X200_1X3_600X200X525P"
+		(property "Footprint" "3_PIN_MALE:HDRV3W60P0X200_1X3_600X200X525P"
 			(at 262.89 120.32 0)
 			(effects
@@
 			)
 		)
-		(property "Value" "10u"
+		(property "Value" "0.1u"
 			(at 120.65 46.9899 90)
 			(effects
@@
 			)
 		)
-		(property "Footprint" "C_Polarized_Tantalum-10uF:CAPPC3528X210N"
+		(property "Footprint" "C_Polarized_Tantalum-10u:CAPPC3528X210N"
 			(at 116.84 46.99 0)
 			(effects
@@
 			)
 		)
-		(property "Footprint" "CAPC2012X145N"
+		(property "Footprint" "C_Ceramic_100n:C0402"
 			(at 163.5 90.17 0)
 			(effects
@@
 			)
 		)
-		(property "Footprint" "C_Ceramic-10uF:C0805"
+		(property "Footprint" "C_Ceramic_100n:C0402"
 			(at 213.03 140.97 0)
 			(effects
@@
 			)
 		)
-		(property "Value" "10u"
+		(property "Value" "0.1u"
 			(at 91.44 46.9899 90)
 			(effects
@@
 			)
 		)
-		(property "Footprint" "C_Polarized_Tantalum-10uF:CAPPC3528X210N"
+		(property "Footprint" "C_Polarized_Tantalum-10u:CAPPC3528X210N"
 			(at 87.63 46.99 0)
 			(effects
@@
 			)
 		)
-		(property "Footprint" "2_pin_Male:HDRV2W60P0X200_1X2_400X200X525P"
+		(property "Footprint" "2_PIN_MALE:HDRV2W60P0X200_1X2_400X200X525P"
 			(at 27.94 -50.47 0)
 			(effects
@@
 			)
 		)
-		(property "Footprint" "C_Ceramic-10uF:C0805"
+		(property "Footprint" "C_Ceramic_100n:C0402"
 			(at 181.61 223.19 0)
 			(effects
@@
 			)
 		)
-		(property "Footprint" ""
+		(property "Footprint" "Resistor_SMD:R_0805_2012Metric_Pad1.20x1.40mm_HandSolder"
 			(at 93.472 99.06 90)
 			(effects
@@
 			)
 		)
-		(property "Footprint" ""
+		(property "Footprint" "2_PIN_MALE:HDRV2W60P0X200_1X2_400X200X525P"
 			(at 95.25 114.3 0)
 			(effects
@@
 			)
 		)
-		(property "Footprint" "CAPC2012X145N"
+		(property "Footprint" "C_Ceramic_100n:C0402"
 			(at 129.21 119.38 0)
 			(effects
@@
 			)
 		)
-		(property "Footprint" "C_Ceramic-100nF:C0402"
+		(property "Footprint" "C_Ceramic_100n:C0402"
 			(at 359.08 114.3 0)
 			(effects
@@
 			)
 		)
-		(property "Footprint" "HDRV3W60P0X200_1X3_600X200X525P"
+		(property "Footprint" "3_PIN_MALE:HDRV3W60P0X200_1X3_600X200X525P"
 			(at 33.02 273.99 0)
 			(effects
@@
 			)
 		)
-		(property "Footprint" "C_Ceramic-10uF:C0805"
+		(property "Footprint" "C_Ceramic_100n:C0402"
 			(at 280.34 95.25 0)
 			(effects
@@
 			)
 		)
-		(property "Footprint" "C_Polarized_Tantalum-10uF:CAPPC3528X210N"
+		(property "Footprint" "C_Polarized_Tantalum-10u:CAPPC3528X210N"
 			(at 80.01 46.99 0)
 			(effects
@@
 			)
 		)
-		(property "Footprint" "830108288709"
+		(property "Footprint" "Crystal16MHZ:830108288709"
 			(at 58.42 101.6 0)
 			(effects
@@
 			)
 		)
-		(property "Footprint" "C_Ceramic-100nF:C0402"
+		(property "Footprint" "C_Ceramic_100n:C0402"
 			(at 305.74 93.98 0)
 			(effects
@@
 			)
 		)
-		(property "Footprint" "HDRV5W64P0X254_1X5_1270X254X610P"
+		(property "Footprint" "5_PIN_MALE:HDRV5W64P0X254_1X5_1270X254X610P"
 			(at 266.7 -33.96 0)
 			(effects
@@
 			)
 		)
-		(property "Footprint" "HDRV3W60P0X200_1X3_600X200X525P"
+		(property "Footprint" "3_PIN_MALE:HDRV3W60P0X200_1X3_600X200X525P"
 			(at 33.02 252.4 0)
 			(effects
@@
 			)
 		)
-		(property "Footprint" "C_Polarized_Tantalum-10uF:CAPPC3528X210N"
+		(property "Footprint" "C_Polarized_Tantalum-10u:CAPPC3528X210N"
 			(at 128.27 46.99 0)
 			(effects
@@
 			)
 		)
-		(property "Footprint" "ESP8266-01_ESP-01:XCVR_ESP8266-01_ESP-01"
+		(property "Footprint" "ESP8266EX:XCVR_ESP8266-01_ESP-01"
 			(at 232.41 114.3 0)
 			(effects
@@
 			)
 		)
-		(property "Footprint" "C0805"
+		(property "Footprint" "C_Ceramic_100n:C0402"
 			(at 313.36 93.98 0)
 			(effects

Commit message: Prva verzija pcb.
Connections:
- no-connect marks 11 -> 13
Changed lines of the file:
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@@
+	)
+	(no_connect
+		(at 171.45 69.85)
+	)
+	(no_connect
+		(at 214.63 111.76)
 	)
 	(no_connect

Commit message: Inicijalno rutiranje, dodani i neki 3d modeli
Parts:
- R1, R2: footprint Resistor_SMD:R_0805_2012Metric_Pad1.20x1.40mm_HandSolder -> Resistor_THT:R_Axial_DIN0204_L3.6mm_D1.6mm_P5.08mm_Horizontal
Changed lines of the file:
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@@
 			)
 		)
-		(property "Footprint" "Resistor_SMD:R_0805_2012Metric_Pad1.20x1.40mm_HandSolder"
+		(property "Footprint" "Resistor_THT:R_Axial_DIN0204_L3.6mm_D1.6mm_P5.08mm_Horizontal"
 			(at 116.84 108.458 90)
 			(effects
@@
 			)
 		)
-		(property "Footprint" "Resistor_SMD:R_0805_2012Metric_Pad1.20x1.40mm_HandSolder"
+		(property "Footprint" "Resistor_THT:R_Axial_DIN0204_L3.6mm_D1.6mm_P5.08mm_Horizontal"
 			(at 93.472 99.06 90)
 			(effects
@@
 					(size 1.27 1.27)
 				)
+				(hide yes)
 			)
 		)

Commit message: Dodani modeli ostalih komponenata u models, Podebljane zice koje nose napajanje, wifi modul okrenut, dodane oznake elemenata
Parts:
- C10, C9: footprint C_Polarized_Tantalum-10u:CAPPC3528X210N -> C_Electrolytic_10uF:CAPPRD200W50D500H1250
- C12, C14, C2, C4, C6: footprint C_Ceramic_100n:C0402 -> C_Ceramic_10u:C0805
- C15, C16: footprint C_Ceramic_100n:C0402 -> C_Ceramic-10pF:CAPC0603X33N
- C7, C8: footprint C_Polarized_Tantalum-10u:CAPPC3528X210N -> C_Electrolytic_0.1uF:CAPAE430X550N
- R1: footprint Resistor_THT:R_Axial_DIN0204_L3.6mm_D1.6mm_P5.08mm_Horizontal -> R_SMD_10kOhm:ERA8KEB1004V
- R2: footprint Resistor_THT:R_Axial_DIN0204_L3.6mm_D1.6mm_P5.08mm_Horizontal -> R_SMD_200Ohm:RESC3216X70N
Other:
- note removed: "Naci na internetu otpornike"
Changed lines of the file:
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@@
 		)
 	)
-	(text "Naci na internetu otpornike"
-		(exclude_from_sim no)
-		(at 127.254 90.17 0)
-		(effects
-			(font
-				(size 1.27 1.27)
-			)
-		)
-	)
 	(text "MICROCONTROLLER"
 		(exclude_from_sim no)
@@
 			)
 		)
-		(property "Footprint" "C_Ceramic_100n:C0402"
+		(property "Footprint" "C_Ceramic_10u:C0805"
 			(at 366.7 114.3 0)
 			(effects
@@
 			)
 		)
-		(property "Footprint" "Resistor_THT:R_Axial_DIN0204_L3.6mm_D1.6mm_P5.08mm_Horizontal"
+		(property "Footprint" "R_SMD_200Ohm:RESC3216X70N"
 			(at 116.84 108.458 90)
 			(effects
@@
 			)
 		)
-		(property "Footprint" "C_Polarized_Tantalum-10u:CAPPC3528X210N"
+		(property "Footprint" "C_Electrolytic_0.1uF:CAPAE430X550N"
 			(at 116.84 46.99 0)
 			(effects
@@
 			)
 		)
-		(property "Footprint" "C_Ceramic_100n:C0402"
+		(property "Footprint" "C_Ceramic-10pF:CAPC0603X33N"
 			(at 163.5 90.17 0)
 			(effects
@@
 			)
 		)
-		(property "Footprint" "C_Ceramic_100n:C0402"
+		(property "Footprint" "C_Ceramic_10u:C0805"
 			(at 213.03 140.97 0)
 			(effects
@@
 			)
 		)
-		(property "Footprint" "C_Polarized_Tantalum-10u:CAPPC3528X210N"
+		(property "Footprint" "C_Electrolytic_0.1uF:CAPAE430X550N"
 			(at 87.63 46.99 0)
 			(effects
@@
 			)
 		)
-		(property "Footprint" "C_Ceramic_100n:C0402"
+		(property "Footprint" "C_Ceramic_10u:C0805"
 			(at 181.61 223.19 0)
 			(effects
@@
 			)
 		)
-		(property "Footprint" "Resistor_THT:R_Axial_DIN0204_L3.6mm_D1.6mm_P5.08mm_Horizontal"
+		(property "Footprint" "R_SMD_10kOhm:ERA8KEB1004V"
 			(at 93.472 99.06 90)
 			(effects
@@
 			)
 		)
-		(property "Footprint" "C_Ceramic_100n:C0402"
+		(property "Footprint" "C_Ceramic-10pF:CAPC0603X33N"
 			(at 129.21 119.38 0)
 			(effects
@@
 			)
 		)
-		(property "Footprint" "C_Ceramic_100n:C0402"
+		(property "Footprint" "C_Ceramic_10u:C0805"
 			(at 280.34 95.25 0)
 			(effects
@@
 			)
 		)
-		(property "Footprint" "C_Polarized_Tantalum-10u:CAPPC3528X210N"
+		(property "Footprint" "C_Electrolytic_10uF:CAPPRD200W50D500H1250"
 			(at 80.01 46.99 0)
 			(effects
@@
 			)
 		)
-		(property "Footprint" "C_Polarized_Tantalum-10u:CAPPC3528X210N"
+		(property "Footprint" "C_Electrolytic_10uF:CAPPRD200W50D500H1250"
 			(at 128.27 46.99 0)
 			(effects
@@
 			)
 		)
-		(property "Footprint" "C_Ceramic_100n:C0402"
+		(property "Footprint" "C_Ceramic_10u:C0805"
 			(at 313.36 93.98 0)
 			(effects

Commit message: Promijenjeni simboli nekih komponenti
Parts:
- C1, C11, C13, C3: footprint C_Ceramic_100n:C0402 -> C0402; symbol CL21X107MRYN3WE:CL21X107MRYN3WE -> C0402C104M4PACTU:C0402C104M4PACTU; Height 1.45 -> 0.55; Manufacturer_Name SAMSUNG -> KEMET; Manufacturer_Part_Number CL21X107MRYN3WE -> C0402C104M4PACTU; Mouser Part Number (none) -> 80-C0402C104M4P; Mouser Price/Stock (none) -> https://www.mouser.co.uk/ProductDetail/KEMET/C0402C104M4PAC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
- C12: footprint C_Ceramic_10u:C0805 -> C0805; Description_1 (none) -> SMD Comm X5R, Ceramic, 10 uF, 20%, 16 VDC, 40 VDC, 85C, -55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
- C15, C16: footprint C_Ceramic-10pF:CAPC0603X33N -> CAPC0603X33N; symbol CL21X107MRYN3WE:CL21X107MRYN3WE -> 02013A100JAT2A:02013A100JAT2A; Description_1 (none) -> Multilayer Ceramic Capacitors MLCC - SMD/SMT 10PF 25volts C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; Height 1.45 -> 0.33; Manufacturer_Name SAMSUNG -> Kyocera AVX; Manufacturer_Part_Number CL21X107MRYN3WE -> 02013A100JAT2A; Mouser Part Number (none) -> 581-02013A100J; Mouser Price/Stock (none) -> https://www.mouser.co.uk/ProductDetail/KYOCERA-AVX/02013A10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
- C5: footprint C_Ceramic_100n:C0402 -> C0402; symbol C0805C106M4PACTU:C0805C106M4PACTU -> C0402C104M4PACTU:C0402C104M4PACTU; Height 1.1 -> 0.55; Manufacturer_Part_Number C0805C106M4PACTU -> C0402C104M4PACTU; Mouser Part Number 80-C0805C106M4P -> 80-C0402C104M4P; Mouser Price/Stock https://www.mouser.co.uk/ProductDetail/KEMET/C0805C106M4PAC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 -> https://www.mouser.co.uk/ProductDetail/KEMET/C0402C104M4PAC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

Commit message: promjena C5.
Parts:
- C5: value 0.1u -> 100n
Changed lines of the file:
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@@
-	)
-	(symbol
-		(lib_id "C0402C104M4PACTU:C0402C104M4PACTU")
-		(at 95.25 133.35 270)
-		(mirror x)
-		(unit 1)
-		(exclude_from_sim no)
-		(in_bom yes)
-		(on_board yes)
-		(dnp no)
-		(property "Reference" "C5"
-			(at 91.44 125.7299 90)
-			(effects
-				(font
-					(size 1.27 1.27)
-				)
-				(justify right)
-			)
-		)
-		(property "Value" "0.1u"
-			(at 91.44 128.2699 90)
-			(effects
-				(font
-					(size 1.27 1.27)
-				)
-				(justify right)
-			)
-		)
-		(property "Footprint" "C0402"
-			(at -0.94 124.46 0)
-			(effects
-				(font
-					(size 1.27 1.27)
-				)
-				(justify left top)
-				(hide yes)
-			)
-		)
-		(property "Datasheet" "https://content.kemet.com/datasheets/KEM_C1006_X5R_SMD.pdf"
-			(at -100.94 124.46 0)
-			(effects
-				(font
-					(size 1.27 1.27)
-				)
-				(justify left top)
-				(hide yes)
-			)
-		)
-		(property "Description" "SMD Comm X5R, Ceramic, 0.1 uF, 20%, 16 VDC, 40 VDC, 85C, -55C, X5R, SMD, MLCC, Temperature Stable, Class II, 5 % , 5 GOhms, 1.21 mg, 0402, 1mm, 0.5mm, 0.5mm, 0.3mm, 0.3mm, 10000, 78  Weeks, 70"
-			(at 95.25 133.35 0)
-			(effects
-				(font
-					(size 1.27 1.27)
-				)
-				(hide yes)
-			)
-		)
-		(property "Height" "0.55"
-			(at -300.94 124.46 0)
-			(effects
-				(font
-					(size 1.27 1.27)
-				)
-				(justify left top)
-				(hide yes)
-			)
-		)
-		(property "Mouser Part Number" "80-C0402C104M4P"
-			(at -400.94 124.46 0)
-			(effects
-				(font
-					(size 1.27 1.27)
-				)
-				(justify left top)
-				(hide yes)
-			)
-		)
-		(property "Mouser Price/Stock" "https://www.mouser.co.uk/ProductDetail/KEMET/C0402C104M4PACTU?qs=K5ytOU5dogo1QkNDOJRLDg%3D%3D"
-			(at -500.94 124.46 0)
-			(effects
-				(font
-					(size 1.27 1.27)
-				)
-				(justify left top)
-				(hide yes)
-			)
-		)
-		(property "Manufacturer_Name" "KEMET"
-			(at -600.94 124.46 0)
-			(effects
-				(font
-					(size 1.27 1.27)
-				)
-				(justify left top)
-				(hide yes)
-			)
-		)
-		(property "Manufacturer_Part_Number" "C0402C104M4PACTU"
-			(at -700.94 124.46 0)
-			(effects
-				(font
-					(size 1.27 1.27)
-				)
-				(justify left top)
-				(hide yes)
-			)
-		)
-		(pin "2"
-		)
-		(pin "1"
-		)
-		(instances
-			(project "schematics"
-				(path "/be652b9a-b406-4c1b-9f3b-1d87964716dc"
-					(reference "C5")
-					(unit 1)
-				)
-			)
-		)
 	)
 	(symbol
@@
 					(unit 1)
 				)
+			)
+		)
+	)
+	(symbol
+		(lib_id "C0402C104M4PACTU:C0402C104M4PACTU")
+		(at 95.25 133.35 90)
+		(unit 1)
+		(exclude_from_sim no)
+		(in_bom yes)
+		(on_board yes)
+		(dnp no)
+		(property "Reference" "C5"
+			(at 91.44 125.7299 90)
+			(effects
+				(font
+					(size 1.27 1.27)
+				)
+				(justify left)
+			)
+		)
+		(property "Value" "100n"
+			(at 91.44 128.2699 90)
+			(effects
+				(font
+					(size 1.27 1.27)
+				)
+				(justify left)
+			)
+		)
+		(property "Footprint" "C0402"
+			(at 191.44 124.46 0)
+			(effects
+				(font
+					(size 1.27 1.27)
+				)
+				(justify left top)
+				(hide yes)
+			)
+		)
+		(property "Datasheet" "https://content.kemet.com/datasheets/KEM_C1006_X5R_SMD.pdf"
+			(at 291.44 124.46 0)
+			(effects
+				(font
+					(size 1.27 1.27)
+				)
+				(justify left top)
+				(hide yes)
+			)
+		)
+		(property "Description" "SMD Comm X5R, Ceramic, 0.1 uF, 20%, 16 VDC, 40 VDC, 85C, -55C, X5R, SMD, MLCC, Temperature Stable, Class II, 5 % , 5 GOhms, 1.21 mg, 0402, 1mm, 0.5mm, 0.5mm, 0.3mm, 0.3mm, 10000, 78  Weeks, 70"
+			(at 95.25 133.35 0)
+			(effects
+				(font
+					(size 1.27 1.27)
+				)
+				(hide yes)
+			)
+		)
+		(property "Height" "0.55"
+			(at 491.44 124.46 0)
+			(effects
+				(font
+					(size 1.27 1.27)
+				)
+				(justify left top)
+				(hide yes)
+			)
+		)
+		(property "Mouser Part Number" "80-C0402C104M4P"
+			(at 591.44 124.46 0)
+			(effects
+				(font
+					(size 1.27 1.27)
+				)
+				(justify left top)
+				(hide yes)
+			)
+		)
+		(property "Mouser Price/Stock" "https://www.mouser.co.uk/ProductDetail/KEMET/C0402C104M4PACTU?qs=K5ytOU5dogo1QkNDOJRLDg%3D%3D"
+			(at 691.44 124.46 0)
+			(effects
+				(font
+					(size 1.27 1.27)
+				)
+				(justify left top)
+				(hide yes)
+			)
+		)
+		(property "Manufacturer_Name" "KEMET"
+			(at 791.44 124.46 0)
+			(effects
+				(font
+					(size 1.27 1.27)
+				)
+				(justify left top)
+				(hide yes)
+			)
+		)
+		(property "Manufacturer_Part_Number" "C0402C104M4PACTU"
+			(at 891.44 124.46 0)
+			(effects
+				(font
+					(size 1.27 1.27)
+				)
+				(justify left top)
+				(hide yes)
+			)
+		)
+		(pin "1"
+		)
+		(pin "2"
+		)
+		(instances
+			(project "schematics"
+				(path "/be652b9a-b406-4c1b-9f3b-1d87964716dc"
+					(reference "C5")
+					(unit 1)
+				)
