File: pcb_design/kicad_schematics/schematics.kicad_pcb (KiCad board)
At the start: 2 copper layers, 57.5 x 33 mm, 29 parts, among them J11 BUTTON-HS-KEY1B, J6 PICKIT, J7 I2C_Communication_Protocol, J8 M22-2510205, J9 SG90, U1 PIC24FJ64GA702-I_SO, U2 ESP8266-01_ESP-01, U3 LM1117LD-3.3, Y2 16MHz crystal

Commit message: Povecan font imena inzenjera
Other:
- board text added: "ColorSorter_A Luka Zeljko Ana Vulin Andjela Savicic"
- board text removed: "ColorSorter_A - Luka Zeljko Ana Vulin Andjela Savicic"
Changed lines of the file:
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@@
 		)
 	)
-	(gr_text "ColorSorter_A\n-\nLuka Zeljko\nAna Vulin\nAndjela Savicic"
-		(at 165.5 79 0)
+	(gr_text "ColorSorter_A\nLuka Zeljko\nAna Vulin\nAndjela Savicic"
+		(at 172.9 80.05 90)
 		(layer "F.SilkS")
 		(effects
 			(font
-				(size 0.75 0.75)
-				(thickness 0.025)
+				(size 1.4 1.4)
+				(thickness 0.3)
 				(bold yes)
 			)

Commit message: Dodane rupe u coskove pcb-a za sarafljenje
Parts:
- moved JP1 2.81 mm to (125.2, 78.0)
- moved J8 1.27 mm to (120.0, 53.1)
- moved U2 0.57 mm to (173.3, 57.8)
Routing:
- net Net-(JP1-A): track 5.80 -> 2.90 mm
- net /MCLR: track 28.0 -> 27.1 mm
- net (no net): vias 0 -> 4
Other:
- board text removed: "BAT"
Changed lines of the file:
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@@
 	(footprint "ESP8266EX:XCVR_ESP8266-01_ESP-01"
 		(layer "F.Cu")
-		(at 173.31 57.23 -90)
+		(at 173.3 57.8 -90)
 		(property "Reference" "U2"
 			(at -4.94 -13.27 90)
@@
 			(polygon
 				(pts
-					(xy 185.66 49.92) (xy 185.66 64.32) (xy 178.96 64.32) (xy 178.96 49.92)
+					(xy 185.65 50.49) (xy 185.65 64.89) (xy 178.95 64.89) (xy 178.95 50.49)
 				)
 			)
@@
 			(polygon
 				(pts
-					(xy 185.66 49.92) (xy 185.66 64.32) (xy 178.96 64.32) (xy 178.96 49.92)
+					(xy 185.65 50.49) (xy 185.65 64.89) (xy 178.95 64.89) (xy 178.95 50.49)
 				)
 			)
@@
 	(footprint "2_PIN_MALE:HDRV2W60P0X200_1X2_400X200X525P"
 		(layer "F.Cu")
-		(at 119.5 52 -90)
+		(at 120.05 53.15 -90)
 		(descr "M22-2510205")
 		(tags "Connector")
@@
 	(footprint "2_PIN_MALE:HDRV2W60P0X200_1X2_400X200X525P"
 		(layer "F.Cu")
-		(at 122.35 77.75 180)
+		(at 125.15 78 180)
 		(descr "M22-2510205")
 		(tags "Connector")
@@
 	)
 	(gr_text "PICKIT"
-		(at 120.5 57 0)
+		(at 121.5 57.15 0)
 		(layer "F.SilkS")
 		(effects
@@
 	)
 	(gr_text "ColorSorter_A\nLuka Zeljko\nAna Vulin\nAndjela Savicic"
-		(at 172.9 80.05 90)
+		(at 170.5 80.3 90)
 		(layer "F.SilkS")
 		(effects
 			(font
-				(size 1.4 1.4)
-				(thickness 0.3)
+				(size 1.3 1.3)
+				(thickness 0.25)
 				(bold yes)
 			)
@@
 	)
 	(gr_text "+"
-		(at 121 54 0)
+		(at 121.8 54.95 0)
 		(layer "F.SilkS")
 		(effects
 			(font
-				(size 0.6 0.6)
-				(thickness 0.1)
+				(size 1 1)
+				(thickness 0.25)
+				(bold yes)
 			)
 		)
@@
 	)
 	(gr_text "JMP_PROG"
-		(at 121 76 0)
+		(at 123.15 76.25 0)
 		(layer "F.SilkS")
 		(effects
@@
 	)
 	(gr_text "-"
-		(at 121 52 0)
+		(at 121.8 53.1 0)
 		(layer "F.SilkS")
 		(effects
 			(font
-				(size 0.6 0.6)
-				(thickness 0.1)
+				(size 1 1)
+				(thickness 0.25)
+				(bold yes)
 			)
 		)
@@
 		)
 	)
-	(gr_text "BAT"
-		(at 119.5 50 0)
-		(layer "F.SilkS")
-		(effects
-			(font
-				(size 0.6 0.6)
-				(thickness 0.1)
-			)
-		)
-	)
 	(gr_text "GND"
 		(at 133.5 80 0)
@@
 		)
 	)
+	(via
+		(at 120.05 50.2)
+		(size 2.2)
+		(drill 2)
+		(layers "F.Cu" "B.Cu")
+		(free yes)
+		(net 0)
+	)
+	(via
+		(at 119.95 78.5)
+		(size 2.2)
+		(drill 2)
+		(layers "F.Cu" "B.Cu")
+		(free yes)
+		(net 0)
+	)
+	(via
+		(at 172.55 50.4)
+		(size 2.2)
+		(drill 2)
+		(layers "F.Cu" "B.Cu")
+		(free yes)
+		(net 0)
+	)
+	(via
+		(at 172.45 78.4)
+		(size 2.2)
+		(drill 2)
+		(layers "F.Cu" "B.Cu")
+		(free yes)
+		(net 0)
+	)
 	(segment
 		(start 147.13 69.825)
@@
 	)
 	(segment
+		(start 162.45 59.07)
+		(end 162.45 61.61)
+		(width 0.5)
+		(layer "F.Cu")
+		(net 2)
+	)
+	(segment
 		(start 128.725 74.5)
 		(end 127.725 73.5)
@@
 	)
 	(segment
-		(start 162.46 58.5)
-		(end 162.46 61.04)
-		(width 0.5)
-		(layer "F.Cu")
-		(net 2)
-	)
-	(segment
 		(start 132.25 75.25)
 		(end 135.5 78.5)
@@
 	)
 	(segment
-		(start 162 58.5)
-		(end 161.55 58.05)
-		(width 0.5)
-		(layer "F.Cu")
-		(net 2)
-	)
-	(segment
 		(start 126.25 61.25)
 		(end 123.33 61.25)
@@
 	)
 	(segment
+		(start 153.5 58.05)
+		(end 161.43 58.05)
+		(width 0.5)
+		(layer "F.Cu")
+		(net 2)
+	)
+	(segment
 		(start 134.35 58)
 		(end 138.05 54.3)
@@
 	)
 	(segment
-		(start 162.46 58.5)
-		(end 162 58.5)
-		(width 0.2)
-		(layer "F.Cu")
-		(net 2)
-	)
-	(segment
 		(start 159.54 78.5)
 		(end 159.54 76.29)
@@
 	)
 	(segment
+		(start 162.45 61.61)
+		(end 161.64 61.61)
+		(width 0.5)
+		(layer "F.Cu")
+		(net 2)
+	)
+	(segment
 		(start 139.7 53.45)
 		(end 139.7 52.65)
@@
 	)
 	(segment
-		(start 162.46 61.04)
-		(end 156.75 66.75)
+		(start 136 74)
+		(end 136.365 73.635)
 		(width 0.5)
 		(layer "F.Cu")
@@
 	)
 	(segment
-		(start 136 74)
-		(end 136.365 73.635)
+		(start 161.64 61.61)
+		(end 156.75 66.5)
 		(width 0.5)
 		(layer "F.Cu")
@@
 	)
 	(segment
-		(start 161.55 58.05)
-		(end 153.5 58.05)
+		(start 161.43 58.05)
+		(end 162.45 59.07)
 		(width 0.5)
 		(layer "F.Cu")
@@
 		(net 2)
 	)
+	(segment
+		(start 156.75 66.5)
+		(end 156.75 66.75)
+		(width 0.5)
+		(layer "F.Cu")
+		(net 2)
+	)
 	(via
 		(at 131.875735 59.124265)
@@
 	)
 	(segment
-		(start 127.8 77.75)
+		(start 125.15 78)
 		(end 128.05 78)
 		(width 0.3)
@@
 	)
 	(segment
-		(start 122.35 77.75)
-		(end 127.8 77.75)
-		(width 0.3)
-		(layer "F.Cu")
-		(net 3)
-	)
-	(segment
 		(start 147.3425 68.3425)
 		(end 149.7575 68.3425)
@@
 	)
 	(segment
-		(start 119.5 54)
-		(end 124.5 54)
-		(width 0.5)
-		(layer "F.Cu")
-		(net 5)
-	)
-	(segment
 		(start 141.5 52)
 		(end 141.5 50.5)
@@
 	)
 	(segment
-		(start 124.5 54)
-		(end 125.5 53)
-		(width 0.5)
-		(layer "F.Cu")
-		(net 5)
-	)
-	(segment
 		(start 125.5 53)
 		(end 129.9 53)
@@
 	)
 	(segment
+		(start 120.05 55.15)
+		(end 123.35 55.15)
+		(width 0.5)
+		(layer "F.Cu")
+		(net 5)
+	)
+	(segment
 		(start 132.81 54.31)
 		(end 132.5 54.31)
@@
 	)
 	(segment
+		(start 123.35 55.15)
+		(end 125.5 53)
+		(width 0.5)
+		(layer "F.Cu")
+		(net 5)
+	)
+	(segment
 		(start 142.5 53)
 		(end 141.5 52)
@@
 	)
 	(segment
-		(start 120.35 77.75)
-		(end 124.275 73.825)
-		(width 0.3)
-		(layer "F.Cu")
-		(net 9)
-	)
-	(segment
 		(start 119 68.670991)
 		(end 119 70)
@@
 	)
 	(segment
-		(start 124.275 73.825)
-		(end 124.275 73.5)
-		(width 0.2)
-		(layer "F.Cu")
-		(net 9)
-	)
-	(segment
 		(start 124.275 73.5)
 		(end 124.275 73.225)
@@
 	)
 	(segment
+		(start 123.15 74.625)
+		(end 124.275 73.5)
+		(width 0.3)
+		(layer "F.Cu")
+		(net 9)
+	)
+	(segment
+		(start 123.15 78)
+		(end 123.15 74.625)
+		(width 0.3)
+		(layer "F.Cu")
+		(net 9)
+	)
+	(segment
 		(start 119.614265 63.845735)
 		(end 119.154265 63.845735)
@@
 	)
 	(segment
-		(start 160.04 66)
-		(end 165 61.04)
+		(start 157 64.5)
+		(end 157.5 64.5)
 		(width 0.3)
 		(layer "F.Cu")
@@
 	)
 	(segment
-		(start 157 64.5)
-		(end 157.5 64.5)
+		(start 160.6 66)
+		(end 164.99 61.61)
 		(width 0.3)
 		(layer "F.Cu")
@@
 	)
 	(segment
+		(start 160.04 66)
+		(end 160.6 66)
+		(width 0.3)
+		(layer "F.Cu")
+		(net 24)
+	)
+	(segment
 		(start 155.975 63.475)
 		(end 147.13 63.475)
@@
 	)
 	(segment
-		(start 146 57.5)
-		(end 151 57.5)
+		(start 154.35 54.15)
+		(end 154.51 53.99)
 		(width 0.3)
 		(layer "F.Cu")
@@
 	)
 	(segment
-		(start 145.745 64.745)
-		(end 147.13 64.745)
+		(start 146 57.5)
+		(end 151 57.5)
 		(width 0.3)
 		(layer "F.Cu")
@@
 	)
 	(segment
-		(start 162.46 53.42)
-		(end 155.731471 53.42)
+		(start 154.51 53.99)
+		(end 162.45 53.99)
 		(width 0.3)
 		(layer "F.Cu")
@@
 	)
 	(segment
-		(start 144.4 63.4)
-		(end 145.745 64.745)
+		(start 145.745 64.745)
+		(end 147.13 64.745)
 		(width 0.3)
 		(layer "F.Cu")
@@
 	)
 	(segment
-		(start 151 57.5)
-		(end 155.08 53.42)
+		(start 144.4 63.4)
+		(end 145.745 64.745)
 		(width 0.3)
 		(layer "F.Cu")
@@
 	)
 	(segment
-		(start 155.08 53.42)
-		(end 155.731471 53.42)
+		(start 151 57.5)
+		(end 154.35 54.15)
 		(width 0.3)
 		(layer "F.Cu")
